File: KiCAD8/ERK01_PWR_Panel.kicad_pcb (KiCad board)
At the start: 2 copper layers, 30 x 128.5 mm, 2 parts

Commit message: JLCPCBに基板製造を発注
Parts:
- removed the G*** at (144.0, 158.0)
- added G***: LOGO, myfootprint:Silk_PNPN_Manufactory_400dpi, F.Cu at (143.5, 155.7)
Other:
- outline, holes or cut-outs redrawn
